Commit message: gazebo7.13

File: urdf/component_snippets.xacro (robot description, xacro)
@@ -17,4 +17,5 @@
 -->
 <robot xmlns:xacro="http://ros.org/wiki/xacro">
+  <xacro:property name="namespace" value="erlecopter" />
   <!-- Macro to add logging to a bag file. -->
   <xacro:macro name="bag_plugin_macro"

File: urdf/erlecopter.xacro (robot description, xacro)
@@ -151,6 +151,5 @@
     sensor_mesh="lidar_lite_v2_withRay/meshes/lidar_lite_v2_withRay.dae">
     <origin xyz="0.13 0.0 0.02" rpy="0 0 0"/>
-  </xacro:sonar_sensor>
--->
+  </xacro:sonar_sensor> -->
   <xacro:include filename="$(find ardupilot_sitl_gazebo_plugin)/urdf/sensors/lidar_sensor.urdf.xacro" />
    <xacro:lidar_sensor

File: urdf/erlecopter_base.xacro (robot description, xacro)
@@ -10,4 +10,5 @@
   <!-- in degrees, 0 so North is towards positive X values, and East is towards negative Y values -->
   <xacro:property name="referenceHeading" value="0" />
+ <xacro:property name="namespace" value="erlecopter" />
   <!--(HS_edit) added namespace uav/ -->
   <!-- Instantiate a controller. -->
